File: trs80-m100.kicad_sch (KiCad schematic)
At the start: 386 parts, among them CN2 A-7224, CN3 TCS-4480, CN4 TCS-4490, CN5 PRINTER CONNECTOR, CN6 RS232C, CN7 LCD-CONN, CN8 LCD-LED-CONN, CN9 3x0.1", CN99 HECO432-01-010, K1 Key_Board, M1 40H373, M10 SystemBus, M11 ROM32k, M12 ROM32k, M13 40H032, M14 40H175, M15 40H244, M16 40H138, M17 40H000, M18 μPD1990AC, M19 80C85, M2 40H245, M20 40H367, M21 40H244, M22 IM6402, M23 40H244, M24 40H032, M25 81C55, M26 40H002, M27 4011, M28 4013, M29 TL064, M3 40H138, M30 TL064, M31 MC14412, M32 40H244, M33 40H157, M34 4584, M35 4584, M36 4013, M4 40H138, M5 40H139, M6 OPTION RAM #3, M7 OPTION RAM #2, M8 OPTION RAM #1, M9 STANDARD RAM, P500 LFIOOKE04Y, P501 LFIOOKE04Y, SW1 SSP32201, SW2 SSB34204, SW3 SLB-22B9-03, SW4 SPJ312U, SW5 SSP32201, T1 2SA1115, T10 2SC2603, T11 2SC2603, T13 2SC2603(E), T14 2SC2603(E), T15 2SC2603(E), T16 2SC2603(E), T17 2SC2603(E), T18 2SC2603, T19 2SA1115, T2 2SC2603, T20 2SC2603, T21 2SC1384(S), T22 2SC2603(E), T23 2SC2603, T24 2SC2603, T25 2SC2603, T27 2SC2603, T28 2SA1115, T3 2SC2603, T4 2SC2603, T5 2SC2603, T6 2SC2603, T7 2SC2603, T8 2SC2603, T9 2SC2603, X1 32.768kHz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

Commit message: Reorganize files then rename project and associated files
Parts:
- C20, C21, C22, C23, C24, C25, C26, C27: symbol trs80-100:C_Tiny -> trs80-m100:C_Tiny
- C52: symbol trs80-100:C_Bipolar -> trs80-m100:C_Bipolar
- C75, C76, C77: symbol trs80-100:C_Bipolar_Small -> trs80-m100:C_Bipolar_Small
- CN2: symbol trs80-100:A-7224 -> trs80-m100:A-7224
- CN3: symbol trs80-100:TCS-4480 -> trs80-m100:TCS-4480
- CN4: symbol trs80-100:TCS-4490 -> trs80-m100:TCS-4490
- CN5: symbol trs80-100:PrinterConn -> trs80-m100:PrinterConn
- CN6: symbol trs80-100:RS232C -> trs80-m100:RS232C
- CN7: symbol trs80-100:LCD-CONN -> trs80-m100:LCD-CONN
- CN8: symbol trs80-100:LCD-LED-CONN -> trs80-m100:LCD-LED-CONN
- CN9: symbol trs80-100:ConnectorSolder-3 -> trs80-m100:ConnectorSolder-3
- D18, D24, D27: symbol trs80-100:surge-absorber -> trs80-m100:surge-absorber
- K1: symbol trs80-100:Key_Board -> trs80-m100:Key_Board
- M1: symbol trs80-100:40H373(1) -> trs80-m100:40H373(1)
- M10: symbol trs80-100:SystemBus -> trs80-m100:SystemBus
- M11, M12: symbol trs80-100:ROM32k -> trs80-m100:ROM32k
- M13, M24: symbol trs80-100:40H032 -> trs80-m100:40H032
- M14: symbol trs80-100:40H175 -> trs80-m100:40H175
- M15: symbol trs80-100:40H244(15) -> trs80-m100:40H244(15)
- M16, M3, M4: symbol trs80-100:40H138 -> trs80-m100:40H138
- M17: symbol trs80-100:40H000 -> trs80-m100:40H000
- M18: symbol trs80-100:μPD1990AC -> trs80-m100:μPD1990AC
- M19: symbol trs80-100:80C85 -> trs80-m100:80C85
- M2: symbol trs80-100:40H245(2) -> trs80-m100:40H245(2)
- M20: symbol trs80-100:40H367 -> trs80-m100:40H367
- M21: symbol trs80-100:40H244(21) -> trs80-m100:40H244(21)
- M22: symbol trs80-100:IM6402 -> trs80-m100:IM6402
- M23: symbol trs80-100:40H244(23) -> trs80-m100:40H244(23)
- M25: symbol trs80-100:81C55 -> trs80-m100:81C55
- M26: symbol trs80-100:40H002 -> trs80-m100:40H002
- M27: symbol trs80-100:4011 -> trs80-m100:4011
- M28: symbol trs80-100:4013-reset-up -> trs80-m100:4013-reset-up
- M31: symbol trs80-100:MC14412 -> trs80-m100:MC14412
- M32: symbol trs80-100:40H244(32) -> trs80-m100:40H244(32)
- M33: symbol trs80-100:40H157 -> trs80-m100:40H157
- M34, M35: symbol trs80-100:4584 -> trs80-m100:4584
- M5: symbol trs80-100:40H139 -> trs80-m100:40H139
- M6, M7, M8, M9: symbol trs80-100:RAM_4x2kiB -> trs80-m100:RAM_4x2kiB
- MR1, MR2, MR3, MR4, MR5, MR6, MR7: symbol trs80-100:R_Network -> trs80-m100:R_Network
- OT2: symbol trs80-100:TN22A -> trs80-m100:TN22A
- RY1: symbol trs80-100:FBR211CD005-M -> trs80-m100:FBR211CD005-M
- RY2: symbol trs80-100:FRL-764D05_1AS-T -> trs80-m100:FRL-764D05_1AS-T
- RY3: symbol trs80-100:FRL-764D05_1BS-T -> trs80-m100:FRL-764D05_1BS-T
- SW1: symbol trs80-100:SW_SSP32201 -> trs80-m100:SW_SSP32201
- SW2: symbol trs80-100:SW_SSB34204 -> trs80-m100:SW_SSB34204
- SW3: symbol trs80-100:SLB-22BP-03 -> trs80-m100:SLB-22BP-03
- SW5: symbol trs80-100:SSP32201 -> trs80-m100:SSP32201
- T1, T19, T28: footprint trs80-100:MitsubishiTransistor_1.25mm -> trs80-m100:MitsubishiTransistor_1.25mm; symbol trs80-100:2SA1115 -> trs80-m100:2SA1115
- T10, T11, T13, T14, T15, T16, T17, T18, T2, T20, T21, T22, T23, T24, T25, T27, T3, T4, T5, T6, T7, T8, T9: footprint trs80-100:MitsubishiTransistor_1.25mm -> trs80-m100:MitsubishiTransistor_1.25mm; symbol trs80-100:2SC2603 -> trs80-m100:2SC2603
